Commit message: Imported upstream version '1.0.2' of 'upstream'

File: urdf/all_sensors.urdf.xacro (robot description, xacro)
@@ -32,4 +32,6 @@
   <!-- KinectV2 -->
   <xacro:include filename="$(find robotnik_sensors)/urdf/kinectv2.urdf.xacro" />
+  <!-- Sick Tim 571 -->
+  <xacro:include filename="$(find robotnik_sensors)/urdf/sick_tim571.urdf.xacro" />
   <!-- Orbbec Astra -->
   <xacro:include filename="$(find robotnik_sensors)/urdf/orbbec_astra.urdf.xacro" />

File: urdf/asus_xtion_pro.urdf.xacro (robot description, xacro)
@@ -7,5 +7,5 @@
   <xacro:property name="asus_xtion_scale" value="1.0"/>
   <xacro:property name="asus_xtion_pro_depth_rel_rgb_py" value="0.0270" />
-  <xacro:property name="asus_xtion_pro_cam_rel_rgb_py"   value="-0.0220" />z
+  <xacro:property name="asus_xtion_pro_cam_rel_rgb_py"   value="-0.0220" />
   <xacro:property name="M_PI" value="3.1415926535897931" />
   <xacro:macro name="sensor_asus_xtion_pro" params="name parent *origin">

File: urdf/kinectv2.urdf.xacro (robot description, xacro)
@@ -2,11 +2,11 @@
 <robot name="sensor_kinectv2" xmlns:xacro="http://ros.org/wiki/xacro">
   <xacro:property name="M_PI" value="3.1415926535897931" />
-	<xacro:property name="cam_px" value="-0.087" />
-	<xacro:property name="cam_py" value="-0.0125" />
-	<xacro:property name="cam_pz" value="0.2870" />
-	<xacro:property name="cam_or" value="0" />
-	<xacro:property name="cam_op" value="0" />
-	<xacro:property name="cam_oy" value="0" />
-  <xacro:macro name="sensor_kinectv2" params="name parent *origin">
+    <xacro:property name="cam_px" value="-0.087" />
+    <xacro:property name="cam_py" value="-0.0125" />
+    <xacro:property name="cam_pz" value="0.2870" />
+    <xacro:property name="cam_or" value="0" />
+    <xacro:property name="cam_op" value="0" />
+    <xacro:property name="cam_oy" value="0" />
+  <xacro:macro name="sensor_kinectv2" params="name parent base:=true *origin">
     <joint name="${name}_rgb_joint" type="fixed">
       <insert_block name="origin" />
@@ -38,5 +38,11 @@
     </link>
   <joint name="${name}_joint" type="fixed">
-    <origin xyz="-0.031 ${-cam_py} -0.016" rpy="0 0 0"/>
+    <!--<origin xyz="-0.031 ${-cam_py} -0.016" rpy="0 0 0"/>--> <!-- with base -->
+    <xacro:if value="${base}">
+        <origin xyz="-0.031 ${-cam_py} -0.016" rpy="0 0 0"/>
+    </xacro:if>
+    <xacro:unless value="${base}">
+        <origin xyz="-0.031 ${-cam_py} -0.016" rpy="0 0 0"/>
+    </xacro:unless>
     <parent link="${name}_rgb_frame"/>
     <child link="${name}_link"/>
@@ -44,15 +50,29 @@
     <link name="${name}_link">
     <visual>
-     <origin xyz="0 0 0" rpy="0 0 ${M_PI/2}"/>
+      <origin xyz="0 0 0" rpy="0 0 ${M_PI/2}"/>
       <geometry>
-       <mesh filename="package://robotnik_sensors/meshes/kinectv2.dae"/>
+        <xacro:if value="${base}">
+          <mesh filename="package://robotnik_sensors/meshes/kinectv2.dae"/>
+        </xacro:if>
+        <xacro:unless value="${base}">
+          <mesh filename="package://robotnik_sensors/meshes/kinectv2_nobase.dae"/>
+        </xacro:unless>
       </geometry>
     </visual>
-	  <collision>
-      <origin xyz="0.0 0.0 0.0" rpy="0 0 0"/>
-	    <geometry>
-	      <box size="0.07271 0.27794 0.073"/>
-	    </geometry>
-	  </collision>
+    <!-- with base -->
+    <collision>
+      <xacro:if value="${base}">
+        <origin xyz="-0.015 0.0 0.03225" rpy="0 0 0"/>
+        <geometry>
+          <box size="0.0943 0.25 0.0645"/>
+        </geometry>
+      </xacro:if>
+      <xacro:unless value="${base}">
+        <origin xyz="-0.015 0.0 0.020" rpy="0 0 0"/>
+        <geometry>
+          <box size="0.0943 0.25 0.045"/>
+        </geometry>
+      </xacro:unless>
+    </collision>
     <inertial>
       <mass value="0.001" />
@@ -66,10 +86,10 @@
        files. However, for Gazebo simulation we need them, so we add them here.
        (Hence, don't publish them additionally!) -->
-	<joint name="${name}_depth_joint" type="fixed">
-	  <origin xyz="0 ${2 * -cam_py} 0" rpy="0 0 0" />
-	  <parent link="${name}_rgb_frame" />
-	  <child link="${name}_depth_frame" />
-	</joint>
-	<link name="${name}_depth_frame">
+    <joint name="${name}_depth_joint" type="fixed">
+      <origin xyz="0 ${2 * -cam_py} 0" rpy="0 0 0" />
+      <parent link="${name}_rgb_frame" />
+      <child link="${name}_depth_frame" />
+    </joint>
+    <link name="${name}_depth_frame">
     <inertial>
       <mass value="0.001" />
@@ -79,11 +99,11 @@
                izz="0.0001" />
     </inertial>
-	</link>
-	<joint name="${name}_depth_optical_joint" type="fixed">
-	  <origin xyz="0 0 0" rpy="${-M_PI/2} 0 ${-M_PI/2}" />
-	  <parent link="${name}_depth_frame" />
-	  <child link="${name}_depth_optical_frame" />
-	</joint>
-	<link name="${name}_depth_optical_frame">
+    </link>
+    <joint name="${name}_depth_optical_joint" type="fixed">
+      <origin xyz="0 0 0" rpy="${-M_PI/2} 0 ${-M_PI/2}" />
+      <parent link="${name}_depth_frame" />
+      <child link="${name}_depth_optical_frame" />
+    </joint>
+    <link name="${name}_depth_optical_frame">
     <inertial>
       <mass value="0.001" />
@@ -93,7 +113,7 @@
                izz="0.0001" />
     </inertial>
-	</link>
-		<!-- Kinect sensor for simulation -->
-	  <sensor_kinectv2_gazebo/>
+    </link>
+        <!-- Kinect sensor for simulation -->
+      <sensor_kinectv2_gazebo/>
   </xacro:macro>
   <xacro:macro name="sensor_kinectv2_gazebo">

File: urdf/orbbec_astra.urdf.xacro (robot description, xacro)
@@ -97,5 +97,5 @@
     </link>
   <!-- RGBD sensor for simulation, same as Kinect -->
-  <sensor_xtion_pro_gazebo/>
+  <sensor_orbbec_astra_gazebo/>
   </xacro:macro>
    <xacro:macro name="sensor_orbbec_astra_gazebo">

File: urdf/sick_s300.urdf.xacro (robot description, xacro)
@@ -12,5 +12,6 @@
 			<geometry>
 				<!--<box size="0.106 0.094 0.152"/>-->
-				<cylinder radius="0.058" length="0.152"/>
+				<!--<cylinder radius="0.058" length="0.152"/>-->
+	     		<mesh filename="package://robotnik_sensors/meshes/sick_s300.dae"/>
 			</geometry>
 		</collision>

File: urdf/sick_s3000.urdf.xacro (robot description, xacro)
@@ -11,5 +11,5 @@
 			<origin xyz="-0.093 0 -0.0625" rpy="0 0 0"/>
 			<geometry>
-				<box size="0.16 0.155 0.211"/>
+	     		<mesh filename="package://robotnik_sensors/meshes/sick_s3000.dae"/>
 			</geometry>
 		</collision>

Commit message: Imported upstream version '1.0.3' of 'upstream'

File: urdf/all_sensors.urdf.xacro (robot description, xacro)
@@ -1,4 +1,4 @@
 <?xml version="1.0"?>
-<robot name="all_sensors" xmlns:xacro="http://ros.org/wiki/xacro">
+<robot name="all_sensors" xmlns:xacro="http://www.ros.org/wiki/xacro">
 	<!-- This file unifies all sensors that can be used on simulation, defined as xacro:macros -->
   <!-- Axis p5512 -->
@@ -36,3 +36,7 @@
   <!-- Orbbec Astra -->
   <xacro:include filename="$(find robotnik_sensors)/urdf/orbbec_astra.urdf.xacro" />
+  <!-- Rplidar -->
+  <xacro:include filename="$(find robotnik_sensors)/urdf/rplidar.urdf.xacro" />
+  <!-- uEye CP Gige -->
+  <xacro:include filename="$(find robotnik_sensors)/urdf/ueye_cp_gige.urdf.xacro" />
 </robot>

File: urdf/asus_xtion_pro.urdf.xacro (robot description, xacro)
@@ -1,4 +1,4 @@
 <?xml version="1.0"?>
-<robot name="sensor_asus_xtion_pro" xmlns:xacro="http://ros.org/wiki/xacro">
+<robot name="sensor_asus_xtion_pro" xmlns:xacro="http://www.ros.org/wiki/xacro">
   <!-- Xacro properties -->
   <!-- xacro:property name="M_SCALE" value="0.001"/ -->
@@ -11,5 +11,5 @@
   <xacro:macro name="sensor_asus_xtion_pro" params="name parent *origin">
     <joint name="${name}_cam_rgb_joint" type="fixed">
-	  <insert_block name="origin" />
+	  <xacro:insert_block name="origin" />
       <parent link="${parent}"/>
       <child link="${name}_cam_rgb_frame" />

File: urdf/axis.urdf.xacro (robot description, xacro)
@@ -1,4 +1,4 @@
 <?xml version="1.0"?>
-<robot name="sensor_axis" xmlns:xacro="http://ros.org/wiki/xacro">
+<robot name="sensor_axis" xmlns:xacro="http://www.ros.org/wiki/xacro">
 	<xacro:property name="ptz_joint_effort_limit" value="100.0" />
   <xacro:property name="ptz_joint_velocity_limit" value="100.0"/>
@@ -12,5 +12,5 @@
 	      <origin xyz="0.180 0.0 0.270"/>
 -->
-				<insert_block name="origin"/>
+				<xacro:insert_block name="origin"/>
 	      <parent link="${parent}"/>
 	      <child link="${name}_link"/>

File: urdf/axis_m5013.urdf.xacro (robot description, xacro)
@@ -1,4 +1,4 @@
 <?xml version="1.0"?>
-<robot name="sensor_axis_m5013" xmlns:xacro="http://ros.org/wiki/xacro">
+<robot name="sensor_axis_m5013" xmlns:xacro="http://www.ros.org/wiki/xacro">
   <xacro:property name="ptz_joint_effort_limit" value="100.0" />
   <xacro:property name="ptz_joint_velocity_limit" value="100.0"/>
@@ -12,5 +12,5 @@
 	      <origin xyz="0.180 0.0 0.270"/>
 -->
-		  <insert_block name="origin"/>
+		  <xacro:insert_block name="origin"/>
 	      <parent link="${parent}"/>
 	      <child link="${name}_link"/>

File: urdf/fotonic.urdf.xacro (robot description, xacro)
@@ -1,7 +1,7 @@
 <?xml version="1.0"?>
-<robot name="sensor_fotonic" xmlns:xacro="http://ros.org/wiki/xacro">
+<robot name="sensor_fotonic" xmlns:xacro="http://www.ros.org/wiki/xacro">
   <xacro:macro name="sensor_fotonic" params="name parent *origin">
     <joint name="${name}_joint" type="fixed">
-			<insert_block name="origin"/>
+			<xacro:insert_block name="origin"/>
       <parent link="${parent}"/>
       <child link="${name}_link"/>

File: urdf/gps.urdf.xacro (robot description, xacro)
@@ -1,9 +1,9 @@
 <?xml version="1.0"?>
-<robot name="sensor_gps" xmlns:xacro="http://ros.org/wiki/xacro">
+<robot name="sensor_gps" xmlns:xacro="http://www.ros.org/wiki/xacro">
   <xacro:macro name="sensor_gps" params="name parent *origin">
 	  <!-- ANTENNA GPS -->
 	  <joint name="${name}_joint" type="fixed">
 	    <axis xyz="0 1 0"/>
-	    <insert_block name="origin"/>
+	    <xacro:insert_block name="origin"/>
 	    <parent link="${parent}"/>
 	    <child link="${name}_link"/>
@@ -40,16 +40,20 @@
 				<updateRate>5.0</updateRate>
 				<bodyName>base_footprint</bodyName>
-				<!-- frameId>base_link</frameId -->
+				<frameId>gps_link</frameId>
 				<topicName>mavros/gps/fix</topicName>
-				<!-- Robotnik position-->
-				<referenceLatitude>39.493800</referenceLatitude>
-				<referenceLongitude>-0.377982</referenceLongitude>
-				<!-- referenceHeading>0</referenceHeading -->
+				<!-- Robotnik position at Fuente del Jarro -->
+				<referenceLatitude>39.5080331</referenceLatitude>
+				<referenceLongitude>-0.4619816</referenceLongitude>
+				<!-- To set heading in ENU orientation (degrees) -->
+				<referenceHeading>90</referenceHeading>
 				<velocityTopicName>fix_velocity</velocityTopicName>
 				<!-- drift>5.0 5.0 5.0</drift -->
-				<drift>0.0001 0.0001 0.0001</drift>
-				<gaussianNoise>0.1 0.1 0.1</gaussianNoise>
-				<velocityDrift>0 0 0</velocityDrift>
-				<velocityGaussianNoise>0.1 0.1 0.1</velocityGaussianNoise>
+				<!--<drift>0.0001 0.0001 0.0001</drift>-->
+				<drift>0.3 0.3 0.3</drift>
+				<!--<gaussianNoise>0.1 0.1 0.1</gaussianNoise>-->
+				<gaussianNoise>0.00001 0.00001 0.00001</gaussianNoise>
+				<velocityDrift>0.00001 0.00001 0.00001</velocityDrift>
+				<!--<velocityGaussianNoise>0.1 0.1 0.1</velocityGaussianNoise>-->
+				<velocityGaussianNoise>0.00001 0.00001 0.00001</velocityGaussianNoise>
       </plugin>
 	</gazebo>

File: urdf/gps_with_mast.urdf.xacro (robot description, xacro)
@@ -1,11 +1,11 @@
 <?xml version="1.0"?>
-<robot name="sensor_gps_with_mast" xmlns:xacro="http://ros.org/wiki/xacro">
-  <property name="mast_height" value="0.5" />
-  <property name="mast_radius" value="0.010" />
+<robot name="sensor_gps_with_mast" xmlns:xacro="http://www.ros.org/wiki/xacro">
+  <xacro:property name="mast_height" value="0.5" />
+  <xacro:property name="mast_radius" value="0.010" />
   <xacro:macro name="sensor_gps_with_mast" params="name parent *origin">
 	  <!-- MAST OF THE ANTENNA GPS -->
 	  <joint name="${name}_joint" type="fixed">
 	    <axis xyz="0 1 0"/>
-	    <insert_block name="origin"/>
+	    <xacro:insert_block name="origin"/>
 	    <parent link="${parent}"/>
 	    <child link="${name}_mast_link"/>

File: urdf/hokuyo3d.urdf.xacro (robot description, xacro)
@@ -1,7 +1,7 @@
 <?xml version="1.0"?>
-<robot name="sensor_hokuyo3d" xmlns:xacro="http://ros.org/wiki/xacro">
+<robot name="sensor_hokuyo3d" xmlns:xacro="http://www.ros.org/wiki/xacro">
   <xacro:macro name="sensor_hokuyo3d" params="name parent *origin">
     <joint name="${name}_laser_fix_joint" type="fixed">
-      <insert_block name="origin" />
+      <xacro:insert_block name="origin" />
       <parent link="${parent}"/>
       <child link="${name}_laser_fix_link"/>

File: urdf/hokuyo_urg04lx.urdf.xacro (robot description, xacro)
@@ -1,4 +1,4 @@
 <?xml version="1.0"?>
-<robot name="sensor_hokuyo_urg04lx" xmlns:xacro="http://ros.org/wiki/xacro">
+<robot name="sensor_hokuyo_urg04lx" xmlns:xacro="http://www.ros.org/wiki/xacro">
   <xacro:macro name="sensor_hokuyo_urg04lx" params="name parent *origin min_angle:=2.0943 max_angle:=-2.0943">
     <joint name="${name}_laser_joint" type="fixed">
@@ -7,5 +7,5 @@
       <!-- TOP MOUNT -->
       <!-- origin xyz="0.0 0.0 0.325"-->
-      <insert_block name="origin" />
+      <xacro:insert_block name="origin" />
       <parent link="${parent}"/>
       <child link="${name}_laser_link"/>

File: urdf/hokuyo_ust10lx.urdf.xacro (robot description, xacro)
@@ -1,7 +1,7 @@
 <?xml version="1.0"?>
-<robot name="sensor_hokuyo_ust10lx" xmlns:xacro="http://ros.org/wiki/xacro">
+<robot name="sensor_hokuyo_ust10lx" xmlns:xacro="http://www.ros.org/wiki/xacro">
   <xacro:macro name="sensor_hokuyo_ust10lx" params="name parent *origin min_angle:=2.3562 max_angle:=-2.3562">
     <joint name="${name}_laser_joint" type="fixed">
-      <insert_block name="origin" />
+      <xacro:insert_block name="origin" />
       <parent link="${parent}"/>
       <child link="${name}_laser_link"/>

File: urdf/hokuyo_utm30lx.urdf.xacro (robot description, xacro)
@@ -1,4 +1,4 @@
 <?xml version="1.0"?>
-<robot name="sensor_hokuyo_utm30lx" xmlns:xacro="http://ros.org/wiki/xacro">
+<robot name="sensor_hokuyo_utm30lx" xmlns:xacro="http://www.ros.org/wiki/xacro">
   <xacro:macro name="sensor_hokuyo_utm30lx" params="name parent *origin min_angle:=2.35 max_angle:=-2.35">
     <joint name="${name}_laser_joint" type="fixed">
@@ -7,5 +7,5 @@
       <!-- TOP MOUNT -->
       <!-- origin xyz="0.0 0.0 0.325"-->
-      <insert_block name="origin" />
+      <xacro:insert_block name="origin" />
       <parent link="${parent}"/>
       <child link="${name}_laser_link"/>

File: urdf/imu.urdf.xacro (robot description, xacro)
@@ -1,9 +1,9 @@
 <?xml version="1.0"?>
-<robot name="sensor_imu" xmlns:xacro="http://ros.org/wiki/xacro">
+<robot name="sensor_imu" xmlns:xacro="http://www.ros.org/wiki/xacro">
   <xacro:macro name="sensor_imu" params="name parent *origin">
 	  <joint name="${name}_joint" type="fixed">
 	      <axis xyz="1 0 0"/>
 	      <!--origin xyz="0 0 0.2825"/-->
-	      <insert_block name="origin"/>
+	      <xacro:insert_block name="origin"/>
 	      <parent link="${parent}"/>
 	      <child link="${name}_link"/>

File: urdf/imu_hector_plugin.urdf.xacro (robot description, xacro)
@@ -1,9 +1,9 @@
 <?xml version="1.0"?>
-<robot name="sensor_imu" xmlns:xacro="http://ros.org/wiki/xacro">
+<robot name="sensor_imu" xmlns:xacro="http://www.ros.org/wiki/xacro">
   <xacro:macro name="sensor_imu_hector" params="name parent *origin">
 	  <joint name="${name}_joint" type="fixed">
 	      <axis xyz="1 0 0"/>
 	      <!--origin xyz="0 0 0.2825"/-->
-	      <insert_block name="origin"/>
+	      <xacro:insert_block name="origin"/>
 	      <parent link="${parent}"/>
 	      <child link="${name}_link"/>
@@ -35,11 +35,23 @@
 	       <updateRate>50.0</updateRate>
 	       <serviceName>imu_service</serviceName>
-	       <accelDrift>0.005 0.005 0.005</accelDrift>
-               <accelGaussianNoise>0.005 0.005 0.005</accelGaussianNoise>
-               <rateDrift>0.02 0.02 0.02</rateDrift>
-               <rateGaussianNoise>0.01 0.01 0.01</rateGaussianNoise>
-	       <headingOffset>0.2</headingOffset>
-               <headingDrift>0.02</headingDrift>
-               <headingGaussianNoise>0.01</headingGaussianNoise>
+	       <!-- orientation parameters -->
+           <yawOffset>0.0</yawOffset>
+           <!--<yawOffset>0.0</yawOffset>-->
+           <yawDrift>0.02</yawDrift>
+           <!--<yawDrift>0.0</yawDrift>-->
+           <yawGaussianNoise>0.01</yawGaussianNoise>
+           <!--<yawGaussianNoise>0.0004</yawGaussianNoise>-->
+           <!-- angular velocities parameters -->
+           <rateOffset>0.0 0.0 0.0</rateOffset>
+           <rateDrift>0.02 0.02 0.02</rateDrift>
+           <!--<rateDrift>0.0 0.0 0.0</rateDrift>-->
+           <rateGaussianNoise>0.01 0.01 0.01</rateGaussianNoise>
+           <!--<rateGaussianNoise>0.004 0.004 0.004</rateGaussianNoise>-->
+           <!-- linear accelerations parameters -->
+           <accelOffset>0.0 0.0 0.0</accelOffset>
+           <accelDrift>0.005 0.005 0.005</accelDrift>
+           <!--<accelDrift>0.0 0.0 0.0</accelDrift>-->
+           <accelGaussianNoise>0.005 0.005 0.005</accelGaussianNoise>
+           <!--<accelGaussianNoise>0.004 0.004 0.004</accelGaussianNoise>-->
 	    </plugin>
 	  </gazebo>

File: urdf/kinect.urdf.xacro (robot description, xacro)
@@ -1,4 +1,4 @@
 <?xml version="1.0"?>
-<robot name="sensor_kinect" xmlns:xacro="http://ros.org/wiki/xacro">
+<robot name="sensor_kinect" xmlns:xacro="http://www.ros.org/wiki/xacro">
   <xacro:property name="M_PI" value="3.1415926535897931" />
 	<xacro:property name="cam_px" value="-0.087" />
@@ -10,5 +10,5 @@
   <xacro:macro name="sensor_kinect" params="name parent *origin">
     <joint name="${name}_rgb_joint" type="fixed">
-      <insert_block name="origin" />
+      <xacro:insert_block name="origin" />
       <parent link="${parent}"/>
       <child link="${name}_rgb_frame" />

File: urdf/kinectv2.urdf.xacro (robot description, xacro)
@@ -1,4 +1,4 @@
 <?xml version="1.0"?>
-<robot name="sensor_kinectv2" xmlns:xacro="http://ros.org/wiki/xacro">
+<robot name="sensor_kinectv2" xmlns:xacro="http://www.ros.org/wiki/xacro">
   <xacro:property name="M_PI" value="3.1415926535897931" />
     <xacro:property name="cam_px" value="-0.087" />
@@ -10,5 +10,5 @@
   <xacro:macro name="sensor_kinectv2" params="name parent base:=true *origin">
     <joint name="${name}_rgb_joint" type="fixed">
-      <insert_block name="origin" />
+      <xacro:insert_block name="origin" />
       <parent link="${parent}"/>
       <child link="${name}_rgb_frame" />

File: urdf/orbbec_astra.urdf.xacro (robot description, xacro)
@@ -1,4 +1,4 @@
 <?xml version="1.0"?>
-<robot name="sensor_orbbec_astra" xmlns:xacro="http://ros.org/wiki/xacro">
+<robot name="sensor_orbbec_astra" xmlns:xacro="http://www.ros.org/wiki/xacro">
   <!-- Xacro properties -->
   <xacro:property name="orbbec_astra_scale" value="1.0"/>
@@ -14,5 +14,5 @@
   <xacro:macro name="sensor_orbbec_astra" params="name parent *origin">
     <joint name="${name}_cam_rgb_joint" type="fixed">
-	  <insert_block name="origin" />
+	  <xacro:insert_block name="origin" />
       <parent link="${parent}"/>
       <child link="${name}_cam_rgb_frame" />

File: urdf/rplidar.urdf.xacro (robot description, xacro)
@@ -1,7 +1,7 @@
 <?xml version="1.0"?>
-<robot xmlns:xacro="http://ros.org/wiki/xacro">
+<robot xmlns:xacro="http://www.ros.org/wiki/xacro">
   <xacro:macro name="sensor_rplidar" params="prefix parent *origin min_angle:=3.14159 max_angle:=-3.14159">
     <joint name="${prefix}_laser_base_joint" type="fixed">
-      <insert_block name="origin" />
+      <xacro:insert_block name="origin" />
       <parent link="${parent}"/>
       <child link="${prefix}_laser_base_link"/>

File: urdf/sick_s300.urdf.xacro (robot description, xacro)
@@ -1,7 +1,7 @@
 <?xml version="1.0"?>
-<robot name="sensor_sick_s300" xmlns:xacro="http://ros.org/wiki/xacro">
+<robot name="sensor_sick_s300" xmlns:xacro="http://www.ros.org/wiki/xacro">
   <xacro:macro name="sensor_sick_s300" params="name parent *origin">
     <joint name="${name}_laser_fix_joint" type="fixed">
-      <insert_block name="origin" />
+      <xacro:insert_block name="origin" />
       <parent link="${parent}"/>
       <child link="${name}_laser_fix_link"/>

File: urdf/sick_s3000.urdf.xacro (robot description, xacro)
@@ -1,7 +1,7 @@
 <?xml version="1.0"?>
-<robot name="sensor_sick_s3000" xmlns:xacro="http://ros.org/wiki/xacro">
+<robot name="sensor_sick_s3000" xmlns:xacro="http://www.ros.org/wiki/xacro">
   <xacro:macro name="sensor_sick_s3000" params="name parent *origin">
     <joint name="${name}_laser_joint" type="fixed">
-      <insert_block name="origin" />
+      <xacro:insert_block name="origin" />
       <parent link="${parent}"/>
       <child link="${name}_laser_link"/>

File: urdf/sick_tim571.urdf.xacro (robot description, xacro)
@@ -1,7 +1,7 @@
 <?xml version="1.0"?>
-<robot xmlns:xacro="http://ros.org/wiki/xacro">
+<robot xmlns:xacro="http://www.ros.org/wiki/xacro">
   <xacro:macro name="sensor_sick_tim571" params="prefix parent *origin min_angle:=-2.36 max_angle:=2.36">
     <joint name="${prefix}laser_base_joint" type="fixed">
-      <insert_block name="origin" />
+      <xacro:insert_block name="origin" />
       <parent link="${parent}"/>
       <child link="${prefix}laser_base_link"/>
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