Commit message: Rebase from 'upstream'

File: urdf/all_sensors.urdf.xacro (robot description, xacro)
@@ -1,4 +1,4 @@
 <?xml version="1.0"?>
-<robot name="all_sensors" xmlns:xacro="http://ros.org/wiki/xacro">
+<robot name="all_sensors" xmlns:xacro="http://www.ros.org/wiki/xacro">
 	<!-- This file unifies all sensors that can be used on simulation, defined as xacro:macros -->
   <!-- Axis p5512 -->
@@ -32,5 +32,11 @@
   <!-- KinectV2 -->
   <xacro:include filename="$(find robotnik_sensors)/urdf/kinectv2.urdf.xacro" />
+  <!-- Sick Tim 571 -->
+  <xacro:include filename="$(find robotnik_sensors)/urdf/sick_tim571.urdf.xacro" />
   <!-- Orbbec Astra -->
   <xacro:include filename="$(find robotnik_sensors)/urdf/orbbec_astra.urdf.xacro" />
+  <!-- Rplidar -->
+  <xacro:include filename="$(find robotnik_sensors)/urdf/rplidar.urdf.xacro" />
+  <!-- uEye CP Gige -->
+  <xacro:include filename="$(find robotnik_sensors)/urdf/ueye_cp_gige.urdf.xacro" />
 </robot>

File: urdf/asus_xtion_pro.urdf.xacro (robot description, xacro)
@@ -1,4 +1,4 @@
 <?xml version="1.0"?>
-<robot name="sensor_asus_xtion_pro" xmlns:xacro="http://ros.org/wiki/xacro">
+<robot name="sensor_asus_xtion_pro" xmlns:xacro="http://www.ros.org/wiki/xacro">
   <!-- Xacro properties -->
   <!-- xacro:property name="M_SCALE" value="0.001"/ -->
@@ -7,9 +7,9 @@
   <xacro:property name="asus_xtion_scale" value="1.0"/>
   <xacro:property name="asus_xtion_pro_depth_rel_rgb_py" value="0.0270" />
-  <xacro:property name="asus_xtion_pro_cam_rel_rgb_py"   value="-0.0220" />z
+  <xacro:property name="asus_xtion_pro_cam_rel_rgb_py"   value="-0.0220" />
   <xacro:property name="M_PI" value="3.1415926535897931" />
   <xacro:macro name="sensor_asus_xtion_pro" params="name parent *origin">
     <joint name="${name}_cam_rgb_joint" type="fixed">
-	  <insert_block name="origin" />
+	  <xacro:insert_block name="origin" />
       <parent link="${parent}"/>
       <child link="${name}_cam_rgb_frame" />

File: urdf/kinectv2.urdf.xacro (robot description, xacro)
@@ -1,14 +1,14 @@
 <?xml version="1.0"?>
-<robot name="sensor_kinectv2" xmlns:xacro="http://ros.org/wiki/xacro">
+<robot name="sensor_kinectv2" xmlns:xacro="http://www.ros.org/wiki/xacro">
   <xacro:property name="M_PI" value="3.1415926535897931" />
-	<xacro:property name="cam_px" value="-0.087" />
-	<xacro:property name="cam_py" value="-0.0125" />
-	<xacro:property name="cam_pz" value="0.2870" />
-	<xacro:property name="cam_or" value="0" />
-	<xacro:property name="cam_op" value="0" />
-	<xacro:property name="cam_oy" value="0" />
-  <xacro:macro name="sensor_kinectv2" params="name parent *origin">
+    <xacro:property name="cam_px" value="-0.087" />
+    <xacro:property name="cam_py" value="-0.0125" />
+    <xacro:property name="cam_pz" value="0.2870" />
+    <xacro:property name="cam_or" value="0" />
+    <xacro:property name="cam_op" value="0" />
+    <xacro:property name="cam_oy" value="0" />
+  <xacro:macro name="sensor_kinectv2" params="name parent base:=true *origin">
     <joint name="${name}_rgb_joint" type="fixed">
-      <insert_block name="origin" />
+      <xacro:insert_block name="origin" />
       <parent link="${parent}"/>
       <child link="${name}_rgb_frame" />
@@ -38,5 +38,11 @@
     </link>
   <joint name="${name}_joint" type="fixed">
-    <origin xyz="-0.031 ${-cam_py} -0.016" rpy="0 0 0"/>
+    <!--<origin xyz="-0.031 ${-cam_py} -0.016" rpy="0 0 0"/>--> <!-- with base -->
+    <xacro:if value="${base}">
+        <origin xyz="-0.031 ${-cam_py} -0.016" rpy="0 0 0"/>
+    </xacro:if>
+    <xacro:unless value="${base}">
+        <origin xyz="-0.031 ${-cam_py} -0.016" rpy="0 0 0"/>
+    </xacro:unless>
     <parent link="${name}_rgb_frame"/>
     <child link="${name}_link"/>
@@ -44,15 +50,29 @@
     <link name="${name}_link">
     <visual>
-     <origin xyz="0 0 0" rpy="0 0 ${M_PI/2}"/>
+      <origin xyz="0 0 0" rpy="0 0 ${M_PI/2}"/>
       <geometry>
-       <mesh filename="package://robotnik_sensors/meshes/kinectv2.dae"/>
+        <xacro:if value="${base}">
+          <mesh filename="package://robotnik_sensors/meshes/kinectv2.dae"/>
+        </xacro:if>
+        <xacro:unless value="${base}">
+          <mesh filename="package://robotnik_sensors/meshes/kinectv2_nobase.dae"/>
+        </xacro:unless>
       </geometry>
     </visual>
-	  <collision>
-      <origin xyz="0.0 0.0 0.0" rpy="0 0 0"/>
-	    <geometry>
-	      <box size="0.07271 0.27794 0.073"/>
-	    </geometry>
-	  </collision>
+    <!-- with base -->
+    <collision>
+      <xacro:if value="${base}">
+        <origin xyz="-0.015 0.0 0.03225" rpy="0 0 0"/>
+        <geometry>
+          <box size="0.0943 0.25 0.0645"/>
+        </geometry>
+      </xacro:if>
+      <xacro:unless value="${base}">
+        <origin xyz="-0.015 0.0 0.020" rpy="0 0 0"/>
+        <geometry>
+          <box size="0.0943 0.25 0.045"/>
+        </geometry>
+      </xacro:unless>
+    </collision>
     <inertial>
       <mass value="0.001" />
@@ -66,10 +86,10 @@
        files. However, for Gazebo simulation we need them, so we add them here.
        (Hence, don't publish them additionally!) -->
-	<joint name="${name}_depth_joint" type="fixed">
-	  <origin xyz="0 ${2 * -cam_py} 0" rpy="0 0 0" />
-	  <parent link="${name}_rgb_frame" />
-	  <child link="${name}_depth_frame" />
-	</joint>
-	<link name="${name}_depth_frame">
+    <joint name="${name}_depth_joint" type="fixed">
+      <origin xyz="0 ${2 * -cam_py} 0" rpy="0 0 0" />
+      <parent link="${name}_rgb_frame" />
+      <child link="${name}_depth_frame" />
+    </joint>
+    <link name="${name}_depth_frame">
     <inertial>
       <mass value="0.001" />
@@ -79,11 +99,11 @@
                izz="0.0001" />
     </inertial>
-	</link>
-	<joint name="${name}_depth_optical_joint" type="fixed">
-	  <origin xyz="0 0 0" rpy="${-M_PI/2} 0 ${-M_PI/2}" />
-	  <parent link="${name}_depth_frame" />
-	  <child link="${name}_depth_optical_frame" />
-	</joint>
-	<link name="${name}_depth_optical_frame">
+    </link>
+    <joint name="${name}_depth_optical_joint" type="fixed">
+      <origin xyz="0 0 0" rpy="${-M_PI/2} 0 ${-M_PI/2}" />
+      <parent link="${name}_depth_frame" />
+      <child link="${name}_depth_optical_frame" />
+    </joint>
+    <link name="${name}_depth_optical_frame">
     <inertial>
       <mass value="0.001" />
@@ -93,7 +113,7 @@
                izz="0.0001" />
     </inertial>
-	</link>
-		<!-- Kinect sensor for simulation -->
-	  <sensor_kinectv2_gazebo/>
+    </link>
+        <!-- Kinect sensor for simulation -->
+      <sensor_kinectv2_gazebo/>
   </xacro:macro>
   <xacro:macro name="sensor_kinectv2_gazebo">

File: urdf/orbbec_astra.urdf.xacro (robot description, xacro)
@@ -1,4 +1,4 @@
 <?xml version="1.0"?>
-<robot name="sensor_orbbec_astra" xmlns:xacro="http://ros.org/wiki/xacro">
+<robot name="sensor_orbbec_astra" xmlns:xacro="http://www.ros.org/wiki/xacro">
   <!-- Xacro properties -->
   <xacro:property name="orbbec_astra_scale" value="1.0"/>
@@ -14,5 +14,5 @@
   <xacro:macro name="sensor_orbbec_astra" params="name parent *origin">
     <joint name="${name}_cam_rgb_joint" type="fixed">
-	  <insert_block name="origin" />
+	  <xacro:insert_block name="origin" />
       <parent link="${parent}"/>
       <child link="${name}_cam_rgb_frame" />
@@ -97,5 +97,5 @@
     </link>
   <!-- RGBD sensor for simulation, same as Kinect -->
-  <sensor_xtion_pro_gazebo/>
+  <sensor_orbbec_astra_gazebo/>
   </xacro:macro>
    <xacro:macro name="sensor_orbbec_astra_gazebo">

File: urdf/sick_s300.urdf.xacro (robot description, xacro)
@@ -1,7 +1,7 @@
 <?xml version="1.0"?>
-<robot name="sensor_sick_s300" xmlns:xacro="http://ros.org/wiki/xacro">
+<robot name="sensor_sick_s300" xmlns:xacro="http://www.ros.org/wiki/xacro">
   <xacro:macro name="sensor_sick_s300" params="name parent *origin">
     <joint name="${name}_laser_fix_joint" type="fixed">
-      <insert_block name="origin" />
+      <xacro:insert_block name="origin" />
       <parent link="${parent}"/>
       <child link="${name}_laser_fix_link"/>
@@ -12,5 +12,6 @@
 			<geometry>
 				<!--<box size="0.106 0.094 0.152"/>-->
-				<cylinder radius="0.058" length="0.152"/>
+				<!--<cylinder radius="0.058" length="0.152"/>-->
+	     		<mesh filename="package://robotnik_sensors/meshes/sick_s300.dae"/>
 			</geometry>
 		</collision>

File: urdf/sick_s3000.urdf.xacro (robot description, xacro)
@@ -1,7 +1,7 @@
 <?xml version="1.0"?>
-<robot name="sensor_sick_s3000" xmlns:xacro="http://ros.org/wiki/xacro">
+<robot name="sensor_sick_s3000" xmlns:xacro="http://www.ros.org/wiki/xacro">
   <xacro:macro name="sensor_sick_s3000" params="name parent *origin">
     <joint name="${name}_laser_joint" type="fixed">
-      <insert_block name="origin" />
+      <xacro:insert_block name="origin" />
       <parent link="${parent}"/>
       <child link="${name}_laser_link"/>
@@ -11,5 +11,5 @@
 			<origin xyz="-0.093 0 -0.0625" rpy="0 0 0"/>
 			<geometry>
-				<box size="0.16 0.155 0.211"/>
+	     		<mesh filename="package://robotnik_sensors/meshes/sick_s3000.dae"/>
 			</geometry>
 		</collision>
